File: hardware/ECAD/SUPERMUSCLE/SUPERMUSCLE.kicad_sch (KiCad schematic)
At the start: 50 parts, among them J1 Conn_01x02_Male, J10 Conn_01x16_Male, J11 Conn_01x05, J12 Conn_Coaxial_Power, J2 Conn_01x02_Male, J3 Conn_01x02_Male, J4 Conn_01x02_Male, J5 Conn_01x02_Male, J6 Conn_01x02_Male, J7 Conn_01x02_Male, J8 Conn_01x02_Male, J9 Conn_01x05, SW1 RotaryEncoder_Switch, SW2 SW_DIP_x01, U1 Teensy4.1, U2 6N138

Commit message: hardware update
Parts:
- added R29: 10K, Resistor_THT:R_Axial_DIN0204_L3.6mm_D1.6mm_P5.08mm_Horizontal, symbol Device:R
- U2: footprint Package_DIP:DIP-14_W7.62mm_Socket_LongPads -> Package_DIP:DIP-8_W7.62mm_Socket_LongPads
Connections:
- net GND: now also R29.1
- net at U2.7 (VO1): now also R29.2
- no-connect marks 53 -> 52
Other:
- moved on the sheet: R27
Changed lines of the file:
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@@
   (junction (at 249.555 28.575) (diameter 0) (color 0 0 0 0)
   )
+  (junction (at 219.075 27.305) (diameter 0) (color 0 0 0 0)
+  )
   (junction (at 245.745 36.195) (diameter 0) (color 0 0 0 0)
   )
@@
   (junction (at 35.56 181.61) (diameter 0) (color 0 0 0 0)
   )
-  (junction (at 220.345 37.465) (diameter 0) (color 0 0 0 0)
-  )
-  (junction (at 220.345 29.845) (diameter 0) (color 0 0 0 0)
-  )
   (junction (at 35.56 160.02) (diameter 0) (color 0 0 0 0)
   )
@@
   (junction (at 45.72 22.86) (diameter 0) (color 0 0 0 0)
   )
+  (junction (at 207.01 29.845) (diameter 0) (color 0 0 0 0)
+  )
   (junction (at 35.56 91.44) (diameter 0) (color 0 0 0 0)
   )
@@
   )
   (junction (at 35.56 22.86) (diameter 0) (color 0 0 0 0)
+  )
+  (junction (at 207.01 37.465) (diameter 0) (color 0 0 0 0)
   )
   (junction (at 45.72 160.02) (diameter 0) (color 0 0 0 0)
@@
   (no_connect (at 259.08 97.79))
   (no_connect (at 229.87 83.82))
-  (no_connect (at 226.695 34.925))
   (no_connect (at 259.08 31.115))
   (no_connect (at 259.08 102.87))
@@
     (stroke (width 0) (type default) (color 0 0 0 0))
   )
+  (wire (pts (xy 207.01 37.465) (xy 207.01 41.91))
+    (stroke (width 0) (type default) (color 0 0 0 0))
+  )
   (wire (pts (xy 114.3 129.54) (xy 142.24 129.54))
     (stroke (width 0) (type default) (color 0 0 0 0))
   )
-  (wire (pts (xy 220.345 37.465) (xy 226.695 37.465))
-    (stroke (width 0) (type default) (color 0 0 0 0))
-  )
   (wire (pts (xy 209.55 78.74) (xy 209.55 109.22))
     (stroke (width 0) (type default) (color 0 0 0 0))
@@
     (stroke (width 0) (type default) (color 0 0 0 0))
   )
+  (wire (pts (xy 207.01 37.465) (xy 226.695 37.465))
+    (stroke (width 0) (type default) (color 0 0 0 0))
+  )
   (wire (pts (xy 116.84 114.3) (xy 142.24 114.3))
     (stroke (width 0) (type default) (color 0 0 0 0))
@@
     (stroke (width 0) (type default) (color 0 0 0 0))
   )
+  (wire (pts (xy 207.01 29.845) (xy 226.695 29.845))
+    (stroke (width 0) (type default) (color 0 0 0 0))
+  )
   (wire (pts (xy 200.025 116.84) (xy 200.025 29.845))
     (stroke (width 0) (type default) (color 0 0 0 0))
@@
     (stroke (width 0) (type default) (color 0 0 0 0))
   )
-  (wire (pts (xy 200.025 29.845) (xy 220.345 29.845))
+  (wire (pts (xy 200.025 29.845) (xy 207.01 29.845))
     (stroke (width 0) (type default) (color 0 0 0 0))
   )
@@
     (stroke (width 0) (type default) (color 0 0 0 0))
   )
+  (wire (pts (xy 219.075 27.305) (xy 226.695 27.305))
+    (stroke (width 0) (type default) (color 0 0 0 0))
+  )
   (wire (pts (xy 259.08 40.005) (xy 253.365 40.005))
     (stroke (width 0) (type default) (color 0 0 0 0))
@@
     (stroke (width 0) (type default) (color 0 0 0 0))
   )
-  (wire (pts (xy 220.345 29.845) (xy 226.695 29.845))
-    (stroke (width 0) (type default) (color 0 0 0 0))
-  )
   (wire (pts (xy 245.745 36.195) (xy 245.745 40.005))
     (stroke (width 0) (type default) (color 0 0 0 0))
@@
     (stroke (width 0) (type default) (color 0 0 0 0))
   )
-  (wire (pts (xy 220.345 37.465) (xy 216.535 37.465))
+  (wire (pts (xy 218.44 27.305) (xy 219.075 27.305))
     (stroke (width 0) (type default) (color 0 0 0 0))
   )
@@
   )
   (wire (pts (xy 58.42 68.58) (xy 114.3 68.58))
+    (stroke (width 0) (type default) (color 0 0 0 0))
+  )
+  (wire (pts (xy 219.075 34.925) (xy 219.075 27.305))
     (stroke (width 0) (type default) (color 0 0 0 0))
   )
@@
     )
   )
-  (symbol (lib_id "Device:R") (at 220.345 33.655 0) (unit 1)
-    (in_bom yes) (on_board yes)
-    (property "Reference" "R27" (id 0) (at 215.0872 33.655 90))
-    (property "Value" "270" (id 1) (at 217.3986 33.655 90))
-    (property "Footprint" "Resistor_THT:R_Axial_DIN0204_L3.6mm_D1.6mm_P5.08mm_Horizontal" (id 2) (at 218.567 33.655 90)
-      (effects (font (size 1.27 1.27)) hide)
-    )
-    (property "Datasheet" "~" (id 3) (at 220.345 33.655 0)
+  (symbol (lib_id "Device:R") (at 207.01 33.655 0) (unit 1)
+    (in_bom yes) (on_board yes)
+    (property "Reference" "R27" (id 0) (at 201.7522 33.655 90))
+    (property "Value" "270" (id 1) (at 204.0636 33.655 90))
+    (property "Footprint" "Resistor_THT:R_Axial_DIN0204_L3.6mm_D1.6mm_P5.08mm_Horizontal" (id 2) (at 205.232 33.655 90)
+      (effects (font (size 1.27 1.27)) hide)
+    )
+    (property "Datasheet" "~" (id 3) (at 207.01 33.655 0)
       (effects (font (size 1.27 1.27)) hide)
     )
@@
     (pin "2")
   )
-  (symbol (lib_id "power:+5V") (at 216.535 37.465 90) (unit 1)
-    (in_bom yes) (on_board yes)
-    (property "Reference" "#PWR027" (id 0) (at 220.345 37.465 0)
-      (effects (font (size 1.27 1.27)) hide)
-    )
-    (property "Value" "+5V" (id 1) (at 213.2838 37.084 90)
+  (symbol (lib_id "power:+5V") (at 207.01 41.91 180) (unit 1)
+    (in_bom yes) (on_board yes)
+    (property "Reference" "#PWR027" (id 0) (at 207.01 38.1 0)
+      (effects (font (size 1.27 1.27)) hide)
+    )
+    (property "Value" "+5V" (id 1) (at 206.629 45.1612 90)
       (effects (font (size 1.27 1.27)) (justify left))
     )
-    (property "Footprint" "" (id 2) (at 216.535 37.465 0)
-      (effects (font (size 1.27 1.27)) hide)
-    )
-    (property "Datasheet" "" (id 3) (at 216.535 37.465 0)
+    (property "Footprint" "" (id 2) (at 207.01 41.91 0)
+      (effects (font (size 1.27 1.27)) hide)
+    )
+    (property "Datasheet" "" (id 3) (at 207.01 41.91 0)
       (effects (font (size 1.27 1.27)) hide)
     )
@@
     (pin "S2")
   )
-  (symbol (lib_id "power:GND") (at 226.695 27.305 270) (unit 1)
-    (in_bom yes) (on_board yes)
-    (property "Reference" "#PWR028" (id 0) (at 220.345 27.305 0)
-      (effects (font (size 1.27 1.27)) hide)
-    )
-    (property "Value" "GND" (id 1) (at 223.4438 27.432 90)
-      (effects (font (size 1.27 1.27)) (justify right))
-    )
-    (property "Footprint" "" (id 2) (at 226.695 27.305 0)
-      (effects (font (size 1.27 1.27)) hide)
-    )
-    (property "Datasheet" "" (id 3) (at 226.695 27.305 0)
+  (symbol (lib_id "power:GND") (at 218.44 27.305 270) (unit 1)
+    (in_bom yes) (on_board yes)
+    (property "Reference" "#PWR028" (id 0) (at 212.09 27.305 0)
+      (effects (font (size 1.27 1.27)) hide)
+    )
+    (property "Value" "GND" (id 1) (at 215.1888 27.432 90)
+      (effects (font (size 1.27 1.27)) (justify right))
+    )
+    (property "Footprint" "" (id 2) (at 218.44 27.305 0)
+      (effects (font (size 1.27 1.27)) hide)
+    )
+    (property "Datasheet" "" (id 3) (at 218.44 27.305 0)
       (effects (font (size 1.27 1.27)) hide)
     )
@@
   (symbol (lib_id "power:GND") (at 246.38 159.385 90) (unit 1)
     (in_bom yes) (on_board yes)
-    (property "Reference" "#PWR?" (id 0) (at 252.73 159.385 0)
+    (property "Reference" "#PWR0108" (id 0) (at 252.73 159.385 0)
       (effects (font (size 1.27 1.27)) hide)
     )
@@
     (property "Reference" "U2" (id 0) (at 234.315 21.0652 0))
     (property "Value" "6N138" (id 1) (at 234.315 23.6021 0))
-    (property "Footprint" "Package_DIP:DIP-14_W7.62mm_Socket_LongPads" (id 2) (at 226.949 24.765 0)
+    (property "Footprint" "Package_DIP:DIP-8_W7.62mm_Socket_LongPads" (id 2) (at 226.949 24.765 0)
       (effects (font (size 1.27 1.27)) hide)
     )
@@
     (pin "8")
   )
+  (symbol (lib_id "Device:R") (at 222.885 34.925 90) (unit 1)
+    (in_bom yes) (on_board yes)
+    (property "Reference" "R29" (id 0) (at 222.885 40.1828 90))
+    (property "Value" "10K" (id 1) (at 222.885 37.8714 90))
+    (property "Footprint" "Resistor_THT:R_Axial_DIN0204_L3.6mm_D1.6mm_P5.08mm_Horizontal" (id 2) (at 222.885 36.703 90)
+      (effects (font (size 1.27 1.27)) hide)
+    )
+    (property "Datasheet" "~" (id 3) (at 222.885 34.925 0)
+      (effects (font (size 1.27 1.27)) hide)
+    )
+    (pin "1")
+    (pin "2")
+  )
   (symbol (lib_id "power:+5V") (at 238.76 159.385 90) (unit 1)
     (in_bom yes) (on_board yes)
-    (property "Reference" "#PWR?" (id 0) (at 242.57 159.385 0)
+    (property "Reference" "#PWR0109" (id 0) (at 242.57 159.385 0)
       (effects (font (size 1.27 1.27)) hide)
     )
@@
     )
     (path "/c23a5fe5-beac-4a0b-8c38-1dd4c4a6cc6a"
-      (reference "#PWR?") (unit 1) (value "GND") (footprint "")
+      (reference "#PWR0108") (unit 1) (value "GND") (footprint "")
     )
     (path "/f0061dc6-6969-4614-ac32-3ad24162f982"
-      (reference "#PWR?") (unit 1) (value "+5V") (footprint "")
+      (reference "#PWR0109") (unit 1) (value "+5V") (footprint "")
     )
     (path "/1ddd64bd-5d76-4fc9-8c5f-fe6a06929ab0"
@@
       (reference "R28") (unit 1) (value "220") (footprint "Resistor_THT:R_Axial_DIN0204_L3.6mm_D1.6mm_P5.08mm_Horizontal")
     )
+    (path "/ccae22b5-2b5c-468a-8dbe-4ff292750326"
+      (reference "R29") (unit 1) (value "10K") (footprint "Resistor_THT:R_Axial_DIN0204_L3.6mm_D1.6mm_P5.08mm_Horizontal")
+    )
     (path "/851aa606-035e-49a9-aeb5-c4e9202d8396"
       (reference "SW1") (unit 1) (value "RotaryEncoder_Switch") (footprint "custom_footprints:5pin_WirePads_RotaryEncoder")
@@
     )
     (path "/cc18fe75-9d0d-40c0-b25a-a8fb54d21ef9"
-      (reference "U2") (unit 1) (value "6N138") (footprint "Package_DIP:DIP-14_W7.62mm_Socket_LongPads")
-    )
-  )
+      (reference "U2") (unit 1) (value "6N138") (footprint "Package_DIP:DIP-8_W7.62mm_Socket_LongPads")
+    )
+  )
